Commit message: Robot arm finished
Something does not work in the gazebo simulation

File: catkin_ws/src/ros_chess/urdf/chess_robot.xacro (robot description, xacro)
@@ -1,119 +1,300 @@
 <?xml version='1.0'?>
 <robot name="chess_arm" xmlns:xacro="http://www.ros.org/wiki/xacro">
-  <link name="base_footprint"></link>
-  <joint name="base_footprint_joint" type="fixed">
-    <origin xyz="0 0 0" rpy="0 0 0" />
-    <parent link="base_footprint"/>
-    <child link="base_link" />
-  </joint>
-  <link name='base_link'>
-    <pose>0 0 0.1 0 0 0</pose>
-    <inertial>
-      <mass value="15.0"/>
-      <origin xyz="0 0 0" rpy="0 0 0"/>
-      <inertia
-          ixx="0.1" ixy="0" ixz="0"
-          iyy="0.1" iyz="0"
-          izz="0.1"
-      />
-    </inertial>
-    <collision name='collision'>
-      <origin xyz="0 0 0" rpy="0 0 0"/>
-      <geometry>
-        <box size=".4 .2 .1"/>
-      </geometry>
-    </collision>
-    <visual name='base_link_visual'>
-      <origin xyz="0 0 0" rpy="0 0 0"/>
-      <geometry>
-        <box size=".4 .2 .1"/>
-      </geometry>
-    </visual>
-    <collision name='rear_caster_collision'>
-      <origin xyz="-0.15 0 -0.05" rpy="0 0 0"/>
-      <geometry>
-        <sphere radius="0.0499"/>
-      </geometry>
-    </collision>
-    <visual name='rear_caster_visual'>
-      <origin xyz="-0.15 0 -0.05" rpy="0 0 0"/>
-      <geometry>
-        <sphere radius="0.05"/>
-      </geometry>
-    </visual>
-    <collision name='front_caster_collision'>
-      <origin xyz="0.15 0 -0.05" rpy="0 0 0"/>
-      <geometry>
-        <sphere radius="0.0499"/>
-      </geometry>
-    </collision>
-    <visual name='front_caster_visual'>
-      <origin xyz="0.15 0 -0.05" rpy="0 0 0"/>
-      <geometry>
-        <sphere radius="0.05"/>
-      </geometry>
-    </visual>
-  </link>
-    <joint type="continuous" name="left_wheel_joint">
-    <origin xyz="0 0.15 0" rpy="0 0 0"/>
-    <child link="left_wheel"/>
+   <!-- Global reference link -->
+  <link name="world"/>
+  <joint name="fixed_base" type="fixed">
+    <parent link="world"/>
+    <child link="base_link"/>
+  </joint>
+  <!-- Arm base link -->
+  <link name="base_link">
+    <inertial>
+      <mass value="5"/>
+      <origin xyz="0.0 0.0 0.0"/>
+      <inertia ixx="0.1135" ixy="0.0" ixz="0.0"
+               iyy="0.1135" iyz="0.0"
+               izz="0.0225"
+      />
+    </inertial>
+    <collision>
+      <geometry>
+        <cylinder radius="0.3" length="0.05"/>
+      </geometry>
+      <origin xyz="0.0 0.0 0.0" rpy="0.0 0.0 0.0"/>
+    </collision>
+    <visual>
+      <geometry>
+        <cylinder radius="0.3" length="0.05"/>
+      </geometry>
+      <material name="grey"/>
+      <origin xyz="0.0 0.0 0.0" rpy="0.0 0.0 0.0"/>
+    </visual>
+  </link>
+  <gazebo reference="base_link">
+    <material>Gazebo/Grey</material>
+  </gazebo>
+  <!-- Shoulder pan joint -->
+  <joint name="1shoulder_pan_joint" type="revolute">
+    <limit lower="-3.14" upper="3.14" effort="100.0" velocity="3.14"/>
     <parent link="base_link"/>
-    <axis xyz="0 1 0" rpy="0 0 0"/>
-    <limit effort="10000" velocity="1000"/>
-    <dynamics damping="1.0" friction="1.0"/>
-  </joint>
-  <link name='left_wheel'>
-    <inertial>
-      <mass value="5.0"/>
-      <origin xyz="0 0 0" rpy="0 1.5707 1.5707"/>
-      <inertia
-          ixx="0.1" ixy="0" ixz="0"
-          iyy="0.1" iyz="0"
-          izz="0.1"
-      />
-    </inertial>
-    <collision name='collision'>
-      <origin xyz="0 0 0" rpy="0 1.5707 1.5707"/>
-      <geometry>
-        <cylinder radius=".1" length=".05"/>
-      </geometry>
-    </collision>
-    <visual name='left_wheel_visual'>
-      <origin xyz="0 0 0" rpy="0 1.5707 1.5707"/>
-      <geometry>
-        <cylinder radius=".1" length=".05"/>
-      </geometry>
-    </visual>
-  </link>
-  <joint type="continuous" name="right_wheel_joint">
-    <origin xyz="0 -0.15 0" rpy="0 0 0"/>
-    <child link="right_wheel"/>
-    <parent link="base_link"/>
-    <axis xyz="0 1 0" rpy="0 0 0"/>
-    <limit effort="10000" velocity="1000"/>
-    <dynamics damping="1.0" friction="1.0"/>
-  </joint>
-  <link name='right_wheel'>
-    <inertial>
-      <mass value="5.0"/>
-      <origin xyz="0 0 0" rpy="0 1.5707 1.5707"/>
-      <inertia
-          ixx="0.1" ixy="0" ixz="0"
-          iyy="0.1" iyz="0"
-          izz="0.1"
-      />
-    </inertial>
-    <collision name='collision'>
-      <origin xyz="0 0 0" rpy="0 1.5707 1.5707"/>
-      <geometry>
-        <cylinder radius=".1" length=".05"/>
-      </geometry>
-    </collision>
-    <visual name='right_wheel_visual'>
-      <origin xyz="0 0 0" rpy="0 1.5707 1.5707"/>
-      <geometry>
-        <cylinder radius=".1" length=".05"/>
-      </geometry>
-    </visual>
-  </link>
-</robot>
+    <child link="shoulder_link"/>
+    <axis xyz="0 0 1"/>
+    <origin xyz="0.0 0.0 0.05" rpy="0.0 0.0 0.0"/>
+    <dynamics damping="0.0" friction="0.0"/>
+  </joint>
+  <!-- Shoulder link -->
+  <link name="shoulder_link">
+    <inertial>
+      <mass value="2"/>
+      <origin xyz="0.0 0.0 0.0" rpy="0.0 0.0 0.0"/>
+      <inertia ixx="0.0317" ixy="0.0" ixz="0.0"
+               iyy="0.0317" iyz="0.0"
+               izz="0.0625"
+      />
+    </inertial>
+    <collision>
+      <geometry>
+        <cylinder radius="0.25" length="0.05"/>
+      </geometry>
+      <origin xyz="0.0 0.0 0.0" rpy="0.0 0.0 0.0"/>
+    </collision>
+    <visual>
+      <geometry>
+        <cylinder radius="0.25" length="0.05"/>
+      </geometry>
+      <material name="orange"/>
+      <origin xyz="0.0 0.0 0.0" rpy="0.0 0.0 0.0"/>
+    </visual>
+  </link>
+  <gazebo reference="shoulder_link">
+    <material>Gazebo/Orange</material>
+  </gazebo>
+  <!-- Shoulder lift joint -->
+  <joint name="2shoulder_lift_joint" type="revolute">
+    <limit lower="-1.5708" upper="1.5708" effort="100" velocity="3.14"/>
+    <parent link="shoulder_link"/>
+    <child link="upper_arm_link"/>
+    <axis xyz="0 1 0"/>
+    <origin xyz="0.0 0.0 0.025" rpy="0.0 0.0 0.0"/>
+    <dynamics damping="0.0" friction="0.0"/>
+  </joint>
+   <!-- Upper arm link -->
+  <link name="upper_arm_link">
+    <inertial>
+      <mass value="3"/>
+      <origin xyz="0.0 0.0 0.1" rpy="0.0 0.0 0.0"/>
+      <inertia ixx="0.2575" ixy="0.0" ixz="0.0"
+               iyy="0.2575" iyz="0.0"
+               izz="0.0150"
+      />
+    </inertial>
+    <collision>
+      <geometry>
+        <cylinder radius="0.1" length="1"/>
+      </geometry>
+      <origin xyz="0.0 0.0 0.5" rpy="0.0 0.0 0.0"/>
+    </collision>
+    <visual>
+      <geometry>
+        <cylinder radius="0.1" length="1"/>
+      </geometry>
+      <material name="orange"/>
+      <origin xyz="0.0 0.0 0.5" rpy="0.0 0.0 0.0"/>
+    </visual>
+  </link>
+  <gazebo reference="upper_arm_link">
+    <material>Gazebo/Orange</material>
+  </gazebo>
+  <!-- Elbow joint -->
+  <joint name="3elbow_joint" type="revolute">
+    <limit lower="-2.3562" upper="2.3562" effort="100" velocity="3.14"/>
+    <parent link="upper_arm_link"/>
+    <child link="forearm_link"/>
+    <axis xyz="0 1 0"/>
+    <origin xyz="0.0 0.0 1" rpy="0.0 0.0 0.0"/>
+    <dynamics damping="0.0" friction="0.0"/>
+  </joint>
+  <!-- Forearm link -->
+  <link name="forearm_link">
+    <inertial>
+      <mass value="2.5"/>
+      <origin xyz="0.0 0.0 0.125" rpy="0.0 0.0 0.0"/>
+      <inertia ixx="0.2146" ixy="0.0" ixz="0.0"
+               iyy="0.2146" iyz="0.0"
+               izz="0.0125"
+      />
+    </inertial>
+    <collision>
+      <geometry>
+        <cylinder radius="0.10" length="1"/>
+      </geometry>
+      <origin xyz="0.0 0.0 0.5" rpy="0.0 0.0 0.0"/>
+    </collision>
+    <visual>
+      <geometry>
+        <cylinder radius="0.10" length="1"/>
+      </geometry>
+      <material name="orange"/>
+      <origin xyz="0.0 0.0 0.5" rpy="0.0 0.0 0.0"/>
+    </visual>
+  </link>
+  <gazebo reference="forearm_link">
+    <material>Gazebo/Orange</material>
+  </gazebo>
+  <!-- Wrist joint -->
+  <joint name="4wrist_joint" type="revolute">
+    <limit lower="-2.3562" upper="2.3562" effort="100" velocity="3.14"/>
+    <parent link="forearm_link"/>
+    <child link="wrist_link"/>
+    <axis xyz="0 1 0"/>
+    <origin xyz="0.0 0.0 1" rpy="0.0 0.0 0.0"/>
+    <dynamics damping="0.0" friction="0.0"/>
+  </joint>
+   <!-- Wrist link -->
+  <link name="wrist_link">
+    <inertial>
+      <mass value="0.1"/>
+      <origin xyz="0.0 0.0 0.05" rpy="0.0 0.0 0.0"/>
+      <inertia ixx="0.00009" ixy="0.0" ixz="0.0"
+               iyy="0.00009" iyz="0.0"
+               izz="0.00002"
+      />
+    </inertial>
+    <collision>
+      <geometry>
+        <cylinder radius="0.05" length="0.2"/>
+      </geometry>
+      <origin xyz="0.0 0.0 0.1" rpy="0.0 0.0 0.0"/>
+    </collision>
+    <visual>
+      <geometry>
+        <cylinder radius="0.05" length="0.2"/>
+      </geometry>
+      <material name="orange"/>
+      <origin xyz="0.0 0.0 0.1" rpy="0.0 0.0 0.0"/>
+    </visual>
+  </link>
+  <gazebo reference="wrist_link">
+    <material>Gazebo/Orange</material>
+  </gazebo>
+  <!-- Gripper base pan joint -->
+  <joint name="5gripper_pan_joint" type="revolute">
+    <limit lower="-3.14" upper="3.14" effort="100" velocity="3.14"/>
+    <parent link="wrist_link"/>
+    <child link="gripper_base_link"/>
+    <axis xyz="0 0 1"/>
+    <origin xyz="0.0 0.0 0.2" rpy="0.0 0.0 0.0"/>
+    <dynamics damping="0.0" friction="0.0"/>
+  </joint>
+  <!-- Gripper base -->
+  <link name="gripper_base_link">
+    <inertial>
+      <mass value="2"/>
+      <origin xyz="0.0 0.0 0.0" rpy="0.0 0.0 0.0"/>
+      <inertia ixx="0.0317" ixy="0.0" ixz="0.0"
+               iyy="0.0317" iyz="0.0"
+               izz="0.0625"
+      />
+    </inertial>
+    <collision>
+      <geometry>
+        <box size=".1 .3 .02"/>
+      </geometry>
+      <origin xyz="0.0 0.0 0.01" rpy="0.0 0.0 0.0"/>
+    </collision>
+    <visual>
+      <geometry>
+        <box size=".1 .3 .02"/>
+      </geometry>
+      <material name="orange"/>
+      <origin xyz="0.0 0.0 0.01" rpy="0.0 0.0 0.0"/>
+    </visual>
+  </link>
+  <gazebo reference="shoulder_link">
+    <material>Gazebo/Orange</material>
+  </gazebo>
+   <!-- Left finger joint -->
+  <joint name="6left_finger_joint" type="prismatic">
+    <limit lower="0" upper="0.13" effort="100.0" velocity="4.0"/>
+    <parent link="gripper_base_link"/>
+    <child link="left_finger"/>
+    <axis xyz="0 1 0"/>
+    <origin xyz="0.0 0.01 0.1" />
+  </joint>
+  <!-- Left finger link -->
+  <link name="left_finger">
+    <inertial>
+      <mass value="0.3"/>
+      <origin xyz="0.0 0.0 0.0" rpy="0.0 0.0 0.0"/>
+      <inertia ixx="0.0009" ixy="0.0" ixz="0.0"
+               iyy="0.0009" iyz="0.0"
+               izz="0.0002"
+      />
+    </inertial>
+    <collision>
+      <geometry>
+        <box size="0.1 0.01 0.2"/>
+      </geometry>
+      <origin xyz="0.0 0.0 0.0" rpy="0.0 0.0 0.0"/>
+    </collision>
+    <visual>
+      <geometry>
+        <box size="0.1 0.01 0.2"/>
+      </geometry>
+      <material name="blue"/>
+      <origin xyz="0.0 0.0 0.0" rpy="0.0 0.0 0.0"/>
+    </visual>
+  </link>
+  <gazebo reference="left_finger">
+    <kp>1000000.0</kp>
+    <kd>100.0</kd>
+    <mu1>15</mu1>
+    <mu2>15</mu2>
+    <fdir1>1 0 0</fdir1>
+    <maxVel>1.0</maxVel>
+    <minDepth>0.002</minDepth>
+    <material>Gazebo/Blue</material>
+  </gazebo>
+  <!-- Right finger joint -->
+  <joint name="7right_finger_joint" type="prismatic">
+    <limit lower="-0.13" upper="0" effort="100.0" velocity="4.0"/>
+    <parent link="gripper_base_link"/>
+    <child link="right_finger"/>
+    <axis xyz="0 1 0"/>
+    <origin xyz="0.0 -0.01 0.1" />
+  </joint>
+  <!-- Right finger link -->
+  <link name="right_finger">
+    <inertial>
+      <mass value="0.3"/>
+      <origin xyz="0.0 0.0 0.0" rpy="0.0 0.0 0.0"/>
+      <inertia ixx="0.0009" ixy="0.0" ixz="0.0"
+               iyy="0.0009" iyz="0.0"
+               izz="0.0002"
+      />
+    </inertial>
+    <collision>
+      <geometry>
+        <box size="0.1 0.01 0.2"/>
+      </geometry>
+      <origin xyz="0.0 0.0 0.0" rpy="0.0 0.0 0.0"/>
+    </collision>
+    <visual>
+      <geometry>
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
Commit message: Robot arm functioning
-Arm_controller
-Modified arm length
-Fixed collision between base and world

File: catkin_ws/src/ros_chess/urdf/chess_robot.xacro (robot description, xacro)
@@ -1,4 +1,10 @@
 <?xml version='1.0'?>
 <robot name="chess_arm" xmlns:xacro="http://www.ros.org/wiki/xacro">
+  <!-- RViz colors -->
+  <xacro:include filename="$(find ros_chess)/urdf/materials.xacro" />
+  <!-- Transmisions -->
+  <xacro:include filename="$(find ros_chess)/urdf/transmission.xacro" />
+  <!-- Gazebo plugin -->
+  <xacro:include filename="$(find ros_chess)/urdf/chess_robot.gazebo" />
    <!-- Global reference link -->
   <link name="world"/>
@@ -35,6 +41,6 @@
   </gazebo>
   <!-- Shoulder pan joint -->
-  <joint name="1shoulder_pan_joint" type="revolute">
-    <limit lower="-3.14" upper="3.14" effort="100.0" velocity="3.14"/>
+  <joint name="J1_shoulder_pan_joint" type="revolute">
+    <limit lower="-3.14" upper="3.14" effort="1000" velocity="3.14"/>
     <parent link="base_link"/>
     <child link="shoulder_link"/>
@@ -71,6 +77,6 @@
   </gazebo>
   <!-- Shoulder lift joint -->
-  <joint name="2shoulder_lift_joint" type="revolute">
-    <limit lower="-1.5708" upper="1.5708" effort="100" velocity="3.14"/>
+  <joint name="J2_shoulder_lift_joint" type="revolute">
+    <limit lower="-1.5708" upper="1.5708" effort="500" velocity="3.14"/>
     <parent link="shoulder_link"/>
     <child link="upper_arm_link"/>
@@ -91,14 +97,14 @@
     <collision>
       <geometry>
-        <cylinder radius="0.1" length="1"/>
-      </geometry>
-      <origin xyz="0.0 0.0 0.5" rpy="0.0 0.0 0.0"/>
-    </collision>
-    <visual>
-      <geometry>
-        <cylinder radius="0.1" length="1"/>
-      </geometry>
-      <material name="orange"/>
-      <origin xyz="0.0 0.0 0.5" rpy="0.0 0.0 0.0"/>
+        <cylinder radius="0.1" length="1.5"/>
+      </geometry>
+      <origin xyz="0.0 0.0 0.75" rpy="0.0 0.0 0.0"/>
+    </collision>
+    <visual>
+      <geometry>
+        <cylinder radius="0.1" length="1.5"/>
+      </geometry>
+      <material name="orange"/>
+      <origin xyz="0.0 0.0 0.75" rpy="0.0 0.0 0.0"/>
     </visual>
   </link>
@@ -107,10 +113,10 @@
   </gazebo>
   <!-- Elbow joint -->
-  <joint name="3elbow_joint" type="revolute">
-    <limit lower="-2.3562" upper="2.3562" effort="100" velocity="3.14"/>
+  <joint name="J3_elbow_joint" type="revolute">
+    <limit lower="-2.3562" upper="2.3562" effort="500" velocity="3.14"/>
     <parent link="upper_arm_link"/>
     <child link="forearm_link"/>
     <axis xyz="0 1 0"/>
-    <origin xyz="0.0 0.0 1" rpy="0.0 0.0 0.0"/>
+    <origin xyz="0.0 0.0 1.5" rpy="0.0 0.0 0.0"/>
     <dynamics damping="0.0" friction="0.0"/>
   </joint>
@@ -127,14 +133,14 @@
     <collision>
       <geometry>
-        <cylinder radius="0.10" length="1"/>
-      </geometry>
-      <origin xyz="0.0 0.0 0.5" rpy="0.0 0.0 0.0"/>
-    </collision>
-    <visual>
-      <geometry>
-        <cylinder radius="0.10" length="1"/>
-      </geometry>
-      <material name="orange"/>
-      <origin xyz="0.0 0.0 0.5" rpy="0.0 0.0 0.0"/>
+        <cylinder radius="0.10" length="1.5"/>
+      </geometry>
+      <origin xyz="0.0 0.0 0.75" rpy="0.0 0.0 0.0"/>
+    </collision>
+    <visual>
+      <geometry>
+        <cylinder radius="0.10" length="1.5"/>
+      </geometry>
+      <material name="orange"/>
+      <origin xyz="0.0 0.0 0.75" rpy="0.0 0.0 0.0"/>
     </visual>
   </link>
@@ -143,10 +149,10 @@
   </gazebo>
   <!-- Wrist joint -->
-  <joint name="4wrist_joint" type="revolute">
-    <limit lower="-2.3562" upper="2.3562" effort="100" velocity="3.14"/>
+  <joint name="J4_wrist_joint" type="revolute">
+    <limit lower="-2.3562" upper="2.3562" effort="200" velocity="3.14"/>
     <parent link="forearm_link"/>
     <child link="wrist_link"/>
     <axis xyz="0 1 0"/>
-    <origin xyz="0.0 0.0 1" rpy="0.0 0.0 0.0"/>
+    <origin xyz="0.0 0.0 1.5" rpy="0.0 0.0 0.0"/>
     <dynamics damping="0.0" friction="0.0"/>
   </joint>
@@ -179,5 +185,5 @@
   </gazebo>
   <!-- Gripper base pan joint -->
-  <joint name="5gripper_pan_joint" type="revolute">
+  <joint name="J5_gripper_pan_joint" type="revolute">
     <limit lower="-3.14" upper="3.14" effort="100" velocity="3.14"/>
     <parent link="wrist_link"/>
@@ -187,8 +193,9 @@
     <dynamics damping="0.0" friction="0.0"/>
   </joint>
+  3
   <!-- Gripper base -->
   <link name="gripper_base_link">
     <inertial>
-      <mass value="2"/>
+      <mass value="0.03"/>
       <origin xyz="0.0 0.0 0.0" rpy="0.0 0.0 0.0"/>
       <inertia ixx="0.0317" ixy="0.0" ixz="0.0"
@@ -215,6 +222,6 @@
   </gazebo>
    <!-- Left finger joint -->
-  <joint name="6left_finger_joint" type="prismatic">
-    <limit lower="0" upper="0.13" effort="100.0" velocity="4.0"/>
+  <joint name="J6_left_finger_joint" type="prismatic">
+    <limit lower="0" upper="0.13" effort="50.0" velocity="4.0"/>
     <parent link="gripper_base_link"/>
     <child link="left_finger"/>
@@ -225,5 +232,5 @@
   <link name="left_finger">
     <inertial>
-      <mass value="0.3"/>
+      <mass value="0.01"/>
       <origin xyz="0.0 0.0 0.0" rpy="0.0 0.0 0.0"/>
       <inertia ixx="0.0009" ixy="0.0" ixz="0.0"
@@ -257,9 +264,9 @@
   </gazebo>
   <!-- Right finger joint -->
-  <joint name="7right_finger_joint" type="prismatic">
-    <limit lower="-0.13" upper="0" effort="100.0" velocity="4.0"/>
+  <joint name="J7_right_finger_joint" type="prismatic">
+    <limit lower="0" upper="0.13" effort="50.0" velocity="4.0"/>
     <parent link="gripper_base_link"/>
     <child link="right_finger"/>
-    <axis xyz="0 1 0"/>
+    <axis xyz="0 -1 0"/>
     <origin xyz="0.0 -0.01 0.1" />
   </joint>
@@ -267,5 +274,5 @@
   <link name="right_finger">
     <inertial>
-      <mass value="0.3"/>
+      <mass value="0.01"/>
       <origin xyz="0.0 0.0 0.0" rpy="0.0 0.0 0.0"/>
       <inertia ixx="0.0009" ixy="0.0" ixz="0.0"

Commit message: TCP point for invese kin and movement node

File: catkin_ws/src/ros_chess/urdf/chess_robot.xacro (robot description, xacro)
@@ -193,5 +193,4 @@
     <dynamics damping="0.0" friction="0.0"/>
   </joint>
-  3
   <!-- Gripper base -->
   <link name="gripper_base_link">
@@ -305,3 +304,29 @@
     <material>Gazebo/Blue</material>
   </gazebo>
+  <!--End effector (TCP) joint-->
+  <joint name="end_effector_joint" type="fixed">
+    <origin xyz="0.0 0.0 0.175" rpy="0 0 0"/>
+    <parent link="gripper_base_link"/>
+    <child link="end_effector_link"/>
+  </joint>
+  <!-- End effector link -->
+  <link name="end_effector_link">
+    <visual>
+      <origin xyz="0 0 0" rpy="0 0 0"/>
+      <geometry>
+        <box size="0.01 0.01 0.01" />
+      </geometry>
+      <material name="red"/>
+     </visual>
+    <inertial>
+      <origin xyz="0 0 0" />
+      <mass value="1.0e-03" />
+      <inertia ixx="1.0e-03" ixy="0.0" ixz="0.0"
+               iyy="1.0e-03" iyz="0.0"
+               izz="1.0e-03" />
+    </inertial>
+  </link>
+  <gazebo reference="end_effector_link">
+    <material>Gazebo/Red</material>
+  </gazebo>
   </robot>
